File: Boards/Panel/panel.sch (EAGLE design)
At the start: 48 parts, among them IC301 MAX232SOIC16, J101 PN61729-S, J401 POWER_IN, J402 OPTRONIK, J403 BUTTON, J404 VIA/JETSON, J405 JOYSTICK, J406 MONITOR, J407 RESV, J408 INDICATOR, T101 MMBT2222A, U201 PSU_5V, U202 PSU_12V, U301 CAN_INTERFACE

Commit message: add extBoard & update panel & motorControl board
> update panel board
> update motorControl board
>add extBoard:
  - to replace mouse movement & left/right click
  - add clear target button
  - add manual lrf value manually using keypad and display it on 4 digits 7-segment
Parts:
- removed C301, C302, C303, C304, C305: 100n, resistor:C-EUC0603
- removed D401: 1N5822, adafruit:DIODESMA
- removed IC301: MAX232SOIC16, SparkFun-DigitalIC:MAX232SOIC16
- removed J406: MONITOR, SparkFun-Connectors:M02-XH-RA
- removed J407: RESV, SparkFun-Connectors:M06-XH-RA
- removed J408: INDICATOR, SparkFun-Connectors:M02-XH-RA
- removed R301: 100, rcl:R-EU_R0603
- removed R302, R306: 100R, rcl:R-EU_R0603
- removed R303, R304, R305: 1k, rcl:R-EU_R0603
- removed R307, R308, R309: 10k, rcl:R-EU_R0603
- removed R401, R402, R403: 1k, resistor:R-EU_R0603
- removed SJ301, SJ302, SJ303, SJ304: (no value), jumper:SJS
- removed SJ401: (no value), jumper:SJ2W
- removed T401, T402: (no value), transistor:MMBT2222ALT1-NPN-SOT23-BEC
- removed U301: CAN_INTERFACE, scorpion:MOD_MCP2515
- added L_DEBUG: (no value), adafruit:LED5MM
- added R101, R4: 100, rcl:R-EU_R0603
- added R102, R103: 1k, resistor:R-EU_R0603
- added R5, R6, R7: 1k, rcl:R-EU_R0603
- added U$2: USB+SHIELD, SparkFun:USB+SHIELD
- added U$3: MOD_MEGA_LAYOUT_SERIAL1, encPhone:MOD_MEGA_LAYOUT_SERIAL1
- added U$4: MOD_MEGA_LAYOUT_SERIAL2, encPhone:MOD_MEGA_LAYOUT_SERIAL2
- added U$5: MOD_MEGA_LAYOUT_SERIAL3, encPhone:MOD_MEGA_LAYOUT_SERIAL3
- added U$6: MOD_MEGA_LAYOUT_ICSP, encPhone:MOD_MEGA_LAYOUT_ICSP
- added U$7: MOD_MEGA_LAYOUT_Y_EVEN, encPhone:MOD_MEGA_LAYOUT_Y_EVEN
- added U1: (no value), scorpion:MOD_MCP2515_NH
- J101: value PN61729-S -> RESV; device con-berg:PN61729-S -> SparkFun-Connectors:M04-XH-RA
- J401: device SparkFun-Connectors:M02-XH-RA -> SparkFun-Connectors:M04-XH-RA
- J403: value BUTTON -> JETSON; device SparkFun-Connectors:M02-XH-RA -> SparkFun-Connectors:M06-XH-RA
- J404: value VIA/JETSON -> JOYSTICK+MONITOR; device SparkFun-Connectors:M08-XH-RA -> SparkFun-Connectors:M04-XH-RA
- J405: value JOYSTICK -> INDICATOR; device SparkFun-Connectors:M04-XH-RA -> SparkFun-Connectors:M02-XH-RA
- U101: value (none) -> MODULE_MEGA2560; device encPhone:MODULE_MEGA -> encPhone:MOD_MEGA_LAYOUT
Connections:
- removed net +12V: J404.2, J405.1, J406.2, SJ401.3, U202.VOUT
- removed net BUS_INT: U101.7, U301.!INT
- removed net INDICATOR: R403.2, U101.13
- removed net JS_PWR_ENABLE: R402.2, U101.8
- removed net MONITOR_PWR_ENABLE: R401.2, U101.53
- removed net N$10: IC301.T1OUT, SJ304.1
- removed net N$2: IC301.R2OUT, SJ301.2
- removed net N$3: IC301.T2OUT, SJ302.1
- removed net N$84: C302.1, IC301.C1-
- removed net N$85: C303.1, IC301.C2-
- removed net N$86: C302.2, IC301.C1+
- removed net N$87: C303.2, IC301.C2+
- removed net N$88: C304.1, IC301.V+
- removed net N$89: C305.1, IC301.V-
- removed net N$9: J406.1, T401.C
- removed net N$95: R304.1, R305.2
- removed net N$96: R301.2, T101.B
- removed net RESV1: U101.6
- removed net RESV2: U101.3
- removed net RESV3: U101.11
- removed net RESV_RX: R307.2, R308.2, SJ304.2
- removed net RESV_TX: IC301.R1IN, R306.1
- removed net SCL: J407.4, U101.21(SCL)
- removed net SDA: J407.3, U101.20(SDA)
- removed net USB_D+: J101.3, U101.USB_D+
- removed net USB_D-: J101.2, U101.USB_D-
- removed net VIA_RX: J404.6, R303.2, R304.2, SJ302.2
- removed net VIA_RXD: IC301.T2IN, R303.1, U101.14(TX3)
- removed net VIA_TX: IC301.R2IN, J404.5, R302.1
- removed net VIA_TXD: R302.2, SJ301.1, U101.15(RX3)
- new net +15V: J403.5, U202.VOUT
- new net INDICATOR_RTN: J405.1, T403.C
- new net JETSON_RX: J403.3, R5.1, R6.1
- new net JETSON_RXD: R5.2, U$4.16(TX2)
- new net JETSON_TX: J403.4, R4.1
- new net JETSON_TXD: R4.2, U$4.17(RX2)
- new net N$14: R6.2, R7.1
- net +24V: now also J402.2, J404.4; no longer D401.C, J402.6
- net BUS_CANH: now also J402.3, J404.2, U1.CAN_H; no longer J402.4, J405.3, U301.CAN_H
- net BUS_CANL: now also J402.4, J404.1, U1.CAN_L; no longer J402.3, J405.4, U301.CAN_L
- net BUS_CS: now also U$7.49, U1.SCK; no longer U101.9, U301.!CS
- net BUTTON_RXD: now also U$3.18(TX1); no longer U101.16(TX2)
- net BUTTON_TX: now also J401.3, R101.1; no longer J403.1, R301.1
- net BUTTON_TXD: now also U$3.19(RX1); no longer U101.17(RX2)
- net GND: now also C203.-, C204.2, J101.2, J403.6, L_DEBUG.C, R7.2, U$2.GND, U$2.P$1, U$2.P$2, U1.VSS, U201.OUT-, U202.GND@1; no longer C301.2, C305.2, IC301.GND, J101.4, J101.S1, J101.S2, J407.5, R305.1, R309.1, U301.VSS
- net MISO: now also U$6.50(MISO), U1.SO; no longer U101.50(MISO), U301.SO
- net MOSI: now also U$6.51(MOSI), U1.SI; no longer U101.51(MOSI, U301.SI
- net N$1: now also R102.1; no longer R403.1
- net N$11: now also L_DEBUG.A, R103.1; no longer R308.1, R309.2
- net N$12: now also R103.2, U$7.*13; no longer D101.A, J101.1
- net N$4: now also U$2.D+, U101.USB_D+; no longer R401.1, T401.B
- net N$5: now also U$2.D-, U101.USB_D-; no longer J405.2, T402.C
- net N$6: now also D101.A, U$2.VBUS; no longer R402.1, T402.B
- net N$7: now also R102.2, U$7.*11; no longer J408.1, T403.C
- net N$8: now also R101.2, T101.B; no longer IC301.R1OUT, SJ303.2
- net RESV_RXD: now also J101.4, U$5.14(TX3); no longer IC301.T1IN, J407.2, R307.1, U101.18(TX1)
- net RESV_TXD: now also J101.3, U$5.15(RX3); no longer J407.1, R306.2, SJ303.1, U101.19(RX1)
- net SCK: now also U$6.52(SCK), U1.!CS; no longer U101.52(SCK), U301.SCK
- net V-: now also J401.4, J402.1, J404.3; no longer C203.-, C204.2, D401.A, J402.5, J403.2, J404.1, T401.E, T402.E, U201.OUT-, U202.GND@1
- net VCC: now also J101.1, J405.2, U1.VDD; no longer C301.1, C304.2, IC301.VCC, J407.6, J408.2, SJ401.1, SJ401.2, U301.VDD
- net VIDEO+: now also J402.5, J403.2; no longer J402.2, J404.7
- net VIDEO-: now also J402.6, J403.1; no longer J402.1, J404.8
