File: Boards/motorControl/motorController.brd (EAGLE design)
At the start: 113 x 75 mm, 92 parts, among them IC301 ATMEGA328P_PDIP, IC401 MAX481CPA, IC402 MAX481CPA, IC403 MCP2515T-I/SO, IC404 MCP2561-E/SN, IC501 PC817, J101 USB+SHIELD, J601 INPUT_PWR, J602 PANEL, J603 OPTRONIK, J604 PAN_PWR, J605 TILT_PWR, J606 TRIGGER, J607 LIMIT_SW, J608 NIX_PAN_COMM, J609 NIX_TILT_COMM, J610 NIX_PAN_IO, J611 NIX_TILT_IO, J612 NIX_PAN_FEEDBACK, J613 PAN_ENCODER/HALL, J614 NIX_TILT_FEEDBACK, J615 TILT_ENCODER/HALL, Q301 16MHz, Q401 16MHz, Q501 IRF1405BV, T501 MMBT2222A, U101 MODULE_MEGA_2560, U201 MP1584_MIN

Commit message: add extBoard & update panel & motorControl board
> update panel board
> update motorControl board
>add extBoard:
  - to replace mouse movement & left/right click
  - add clear target button
  - add manual lrf value manually using keypad and display it on 4 digits 7-segment
Parts:
- removed C204, C305: 100n, resistor:C0603
- removed C401, C402: 100n, rcl:C0603
- removed C403, C404: 22p, rcl:C0603
- removed C601: 470uF/50V, resistor:E5-10,5
- removed D401: 1N4004, adafruit:SOD-323F
- removed IC301: ATMEGA328P_PDIP, SparkFun-DigitalIC:DIL28-3
- removed J102: (no value), SparkFun-Connectors:MOLEX-1X2
- removed J602: PANEL, SparkFun-Connectors:XH-4-RA
- removed J612: NIX_PAN_FEEDBACK, SparkFun-Connectors:XH-6-RA
- removed J613: PAN_ENCODER/HALL, SparkFun-Connectors:MOLEX-1X6
- removed J614: NIX_TILT_FEEDBACK, SparkFun-Connectors:XH-6-RA
- removed J615: TILT_ENCODER/HALL, SparkFun-Connectors:MOLEX-1X6
- removed LD401: YELLOW, led:LED5MM
- removed Q301, Q401: 16MHz, special:QS
- removed R301, R405, R605, R607, R609, R611, R613, R615: 10k, rcl:R0603
- removed R606, R608, R610, R612, R614, R616: 100, rcl:R0603
- added C201: 470uF/50V, resistor:E5-10,5
- added C202: 100uF/25V, resistor:E5-10,5
- added D603, D604: 1N5817, adafruit:SOD-323F
- added IC305: MCP2515T-I/SO, microchip:SO-18
- added IC306: MCP2561-E/SN, microchip:SOIC-8
- added R305: 10k, rcl:R0603
- added R306: 120R, rcl:R0603
- added U$10: MOD_MEGA_LAYOUT_I2C, encPhone:MOD_MEGA_LAYOUT_I2C
- added U$8: MOD_MEGA_LAYOUT_Y_ODD, encPhone:MOD_MEGA_LAYOUT_Y_ODD
- added UART_RESV: (no value), SparkFun-Connectors:1X03_LOCK
- added X301: 16MHz, special:QS
- C203: value 100uF/25V -> 100n; device resistor:E5-10,5 -> resistor:C0603
- C301: value 22p -> 100n; device resistor:C0603 -> rcl:C0603
- C304: device resistor:C0603 -> rcl:C0603
- IC403: value MCP2515T-I/SO -> MAX481CPA; device microchip:SO-18 -> maxim:DIL08
- IC404: value MCP2561-E/SN -> MAX481CPA; device microchip:SOIC-8 -> maxim:DIL08
- J601: value INPUT_PWR -> PANEL; device SparkFun-Connectors:XH-4-RA -> SparkFun-Connectors:XH-8-RA
- R403: value 120R -> 120
- R404: value 330R -> 120; device resistor:R0603 -> rcl:R0603
- U$7: value MOD_MEGA_LAYOUT_Z_ODD -> MOD_MEGA_LAYOUT_Y_EVEN; device encPhone:MOD_MEGA_LAYOUT_Z_ODD -> encPhone:MOD_MEGA_LAYOUT_Y_EVEN
- U$9: value MOD_MEGA_LAYOUT_Y_ODD -> MOD_MEGA_LAYOUT_Z_ODD; device encPhone:MOD_MEGA_LAYOUT_Y_ODD -> encPhone:MOD_MEGA_LAYOUT_Z_ODD
- moved J609 201.4 mm to (-92.1, 57.8), turned to 90 degrees
- moved J608 197.6 mm to (-92.1, 43.8), turned to 90 degrees
- moved R402 195.4 mm to (-94.3, 46.4), turned to 270 degrees
- moved R401 194.6 mm to (-94.3, 41.3), turned to 270 degrees
- moved SJ201 182.0 mm to (-96.2, 36.4), turned to 90 degrees
- moved R403 180.5 mm to (-94.3, 55.2), turned to 270 degrees
- moved IC404 168.3 mm to (-82.5, 56.5), flipped to the top, turned to 90 degrees
- moved R404 150.3 mm to (-94.3, 60.3)
- moved IC403 149.7 mm to (-82.5, 46.4), flipped to the top, turned to 90 degrees
- moved SJ202 148.4 mm to (-63.9, 19.8), turned to 135 degrees
- moved IC402 141.8 mm to (-47.6, 36.5), turned to 180 degrees
- moved J101 131.8 mm to (-16.2, 8.57), turned to 90 degrees
- moved IC401 131.5 mm to (-37.5, 36.5), turned to 180 degrees
- moved C602 128.5 mm to (-80.6, 5.08)
- moved J605 125.3 mm to (-88.3, 5.08), turned to 90 degrees
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Connections:
- net MTR_RXD renamed MTR_PAN_RXD
- net MTR_TXD renamed MTR_PAN_TXD
- removed net !RESET1: C301.1, D301.A, IC301.1, R301.1
- removed net CAN_CS: IC403.16
- removed net CAN_INT: IC403.12, LD401.K
- removed net FEED_RXD: IC301.2, U$6.Z10
- removed net FEED_TXD: IC301.3, U$6.Z9
- removed net N$21: C401.1, D401.A, IC403.17, R405.1
- removed net N$22: C403.2, IC403.8, Q401.1
- removed net N$23: C404.2, IC403.7, Q401.2
- removed net N$24: LD401.A, R404.2
- removed net N$5: C303.2, IC301.10, Q301.1
- removed net P_FEED1: IC301.4, J612.3, R606.1
- removed net P_FEED2: IC301.28, J612.2, R608.1
- removed net P_FEED3: IC301.27, J612.1, R610.1
- removed net P_HALL1/A: J613.3, R605.1, R606.2
- removed net P_HALL2/B: J613.4, R607.1, R608.2
- removed net P_HALL3/Z: J613.5, R609.1, R610.2
- removed net P_VDD: J612.6, J613.6, R605.2, R607.2, R609.2
- removed net RX+: IC401.6, J608.2, J609.2, R401.1
- removed net RX-: IC401.7, J608.1, J609.1, R401.2
- removed net TX+: IC402.6, J608.4, J609.4, R402.1
- removed net TX-: IC402.7, J608.3, J609.3, R402.2
- removed net T_FEED1: IC301.5, J614.3, R616.1
- removed net T_FEED2: IC301.26, J614.2, R614.1
- removed net T_FEED3: IC301.25, J614.1, R612.1
- removed net T_HALL1/A: J615.3, R615.1, R616.2
- removed net T_HALL2/B: J615.4, R613.1, R614.2
- removed net T_HALL3/Z: J615.5, R611.1, R612.2
- removed net T_VDD: J614.6, J615.6, R611.2, R613.2, R615.2
- new net !CAN_CS: IC305.16, U$7.Y6
- new net +24V: C201.+, D201.C, J601.5, J601.6, J603.2, U201.1
- new net MTR_TILT_RXD: IC403.4, U$6.Z10
- new net MTR_TILT_TXD: IC404.1, U$6.Z9
- new net N$12: D604.C, J611.1
- new net N$13: C302.2, IC305.8, X301.1
- new net PAN_RX+: IC401.6, J608.2, R401.1
- new net PAN_RX-: IC401.7, J608.1, R401.2
- new net PAN_TX+: IC402.6, J608.4, R402.1
- new net PAN_TX-: IC402.7, J608.3, R402.2
- new net P_RESV: D603.A, U$9.Z7
- new net RXD2: U$5.X8, UART_RESV.1
- new net SCL: U$10.Y14
- new net SDA: U$10.Y13
- new net TILT_RX+: IC403.6, J609.2, R403.1
- new net TILT_RX-: IC403.7, J609.1, R403.2
- new net TILT_TX+: IC404.6, J609.4, R404.1
- new net TILT_TX-: IC404.7, J609.3, R404.2
- new net TXD2: U$5.X5, UART_RESV.2
- new net T_RESV: D604.A, U$8.Y11
- net CAN_H: now also IC306.7, J601.1, J603.6, R306.2; no longer IC404.7, J602.1, J603.4, R403.2
- net CAN_L: now also IC306.6, J601.2, J603.5, R306.1; no longer IC404.6, J602.2, J603.3, R403.1
- net GND: now also C202.-, C203.2, C304.2, IC305.9, IC306.2, IC306.8, IC403.5, IC404.3, IC404.5, J607.4, UART_RESV.3; no longer C203.-, C204.2, C304.1, C305.2, C401.2, C402.2, C403.1, C404.1, IC301.22, IC301.8, IC403.9, IC404.8, J607.1, J610.1, J611.1, J612.4, J612.5, J613.1, J613.2, J614.4, J614.5, J615.1, J615.2
- net MISO: now also IC305.15; no longer IC403.15
- net MOSI: now also IC305.14; no longer IC403.14
- net N$10: now also U$7.Y8; no longer J102.1, U$5.X8
- net N$11: now also D603.C, J610.1; no longer J102.2, U$5.X5
- net N$14: now also C303.2, IC305.7, X301.2; no longer C304.2, IC301.21
- net N$6: now also R101.1, U$7.Y4; no longer C302.2, IC301.9, Q301.2
- net N$9: now also C301.1, D301.A, IC305.17, R305.1; no longer R101.1, U$7.Z7
- net P_ENABLE: now also U$9.Z5; no longer U$9.Y11
- net P_FAULT_RESET: now also U$9.Z3; no longer U$9.Y9
- net P_HEALTH: now also U$9.Z1; no longer U$9.Y7
- net P_HOME_SWITCH: now also J607.3, U$7.Y2; no longer J607.2, U$7.Z5
- net RXCAN: now also IC305.2, IC306.4; no longer IC403.2, IC404.4
- net SCK: now also IC305.13; no longer IC403.13
- net TRIGGER_PWM: now also U$7.Y10
- net TRIGGER_PWR_EN: now also U$7.Y12
- net TXCAN: now also IC305.1, IC306.1; no longer IC403.1, IC404.1
- net T_DOWN_LIM: now also J607.1, U$8.Y3; no longer J607.4, U$7.Z1
- net T_ENABLE: now also U$8.Y9; no longer U$9.Y5
- net T_FAULT_RESET: now also U$8.Y7; no longer U$9.Y3
- net T_HEALTH: now also U$8.Y5; no longer U$9.Y1
- net T_UP_LIM: now also J607.2, U$8.Y1; no longer J607.3, U$7.Z3
- net V+: no longer C601.+, D201.C, J601.1, J601.2, J603.6, U201.1
- net V-: now also C201.-, J601.7, J601.8, J603.1; no longer C601.-, J601.3, J601.4, J603.5
- net VCC: now also C202.+, C203.1, C304.1, IC305.18, IC306.3, IC403.2, IC403.3, IC403.8, IC404.8, R305.2; no longer C203.+, C204.1, C305.1, C402.1, D401.C, IC301.20, IC301.7, IC403.18, IC404.3, R301.2, R404.1, R405.2
- net VIDEO+: now also J601.3, J603.4; no longer J602.3, J603.2
- net VIDEO-: now also J601.4, J603.3; no longer J602.4, J603.1
Routing:
- net GND: track 572.0 -> 382.8 mm, vias 0 -> 2
- net VCC: track 183.9 -> 277.2 mm, vias 0 -> 2
- net V-: track 181.2 -> 92.9 mm
- net PAN_RX-: track 0.00 -> 68.1 mm
- net PAN_RX+: track 0.00 -> 66.5 mm
- net N$7: track 13.0 -> 74.4 mm
- net PAN_TX-: track 0.00 -> 59.4 mm
- net PAN_TX+: track 0.00 -> 58.4 mm
- net P_FEED1: track 54.3 -> 0.00 mm
- net TRIGGER_PWM: track 0.00 -> 54.2 mm
- net +24V: track 0.00 -> 52.6 mm
- net V+: track 110.2 -> 57.6 mm
- net TRIGGER_PWR_EN: track 0.00 -> 52.6 mm
- net P_FEED3: track 51.0 -> 0.00 mm
- net T_FEED1: track 49.5 -> 0.00 mm
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Other:
- board size 113 x 75 mm -> 100 x 65 mm
- board text added: "RWS-motorController_20180412"
- board text removed: "RWS-motorDriver_20180119"
