File: Boards/motorControl/motorController.sch (EAGLE design)
At the start: 92 parts, among them IC301 ATMEGA328P_PDIP, IC401 MAX481CPA, IC402 MAX481CPA, IC403 MCP2515T-I/SO, IC404 MCP2561-E/SN, IC501 PC817, J101 USB+SHIELD, J601 INPUT_PWR, J602 PANEL, J603 OPTRONIK, J604 PAN_PWR, J605 TILT_PWR, J606 TRIGGER, J607 LIMIT_SW, J608 NIX_PAN_COMM, J609 NIX_TILT_COMM, J610 NIX_PAN_IO, J611 NIX_TILT_IO, J612 NIX_PAN_FEEDBACK, J613 PAN_ENCODER/HALL, J614 NIX_TILT_FEEDBACK, J615 TILT_ENCODER/HALL, Q301 16MHz, Q401 16MHz, Q501 IRF1405BV, T501 MMBT2222A, U101 MODULE_MEGA_2560, U201 MP1584_MIN

Commit message: add extBoard & update panel & motorControl board
> update panel board
> update motorControl board
>add extBoard:
  - to replace mouse movement & left/right click
  - add clear target button
  - add manual lrf value manually using keypad and display it on 4 digits 7-segment
Parts:
- removed C204, C305: 100n, resistor:C-EUC0603
- removed C401, C402: 100n, rcl:C-EUC0603
- removed C403, C404: 22p, rcl:C-EUC0603
- removed C601: 470uF/50V, resistor:CPOL-EUE5-10.5
- removed D401: 1N4004, adafruit:DIODESOD-323F
- removed IC301: ATMEGA328P_PDIP, SparkFun-DigitalIC:ATMEGA328P_PDIP
- removed J102: (no value), SparkFun-Connectors:M02POLAR
- removed J602: PANEL, SparkFun-Connectors:M04-XH-RA
- removed J612: NIX_PAN_FEEDBACK, SparkFun-Connectors:M06-XH-RA
- removed J613: PAN_ENCODER/HALL, SparkFun-Connectors:M06POLAR
- removed J614: NIX_TILT_FEEDBACK, SparkFun-Connectors:M06-XH-RA
- removed J615: TILT_ENCODER/HALL, SparkFun-Connectors:M06POLAR
- removed LD401: YELLOW, led:LED5MM
- removed Q301, Q401: 16MHz, special:XTAL/S
- removed R301, R405, R605, R607, R609, R611, R613, R615: 10k, rcl:R-EU_R0603
- removed R606, R608, R610, R612, R614, R616: 100, rcl:R-EU_R0603
- added C201: 470uF/50V, resistor:CPOL-EUE5-10.5
- added C202: 100uF/25V, resistor:CPOL-EUE5-10.5
- added D603, D604: 1N5817, adafruit:DIODESOD-323F
- added IC305: MCP2515T-I/SO, microchip:MCP2515T-I/SO
- added IC306: MCP2561-E/SN, microchip:MCP2561-E/SN
- added R305: 10k, rcl:R-EU_R0603
- added R306: 120R, rcl:R-EU_R0603
- added U$10: MOD_MEGA_LAYOUT_I2C, encPhone:MOD_MEGA_LAYOUT_I2C
- added U$8: MOD_MEGA_LAYOUT_Y_ODD, encPhone:MOD_MEGA_LAYOUT_Y_ODD
- added UART_RESV: (no value), SparkFun-Connectors:M03LOCK
- added X301: 16MHz, special:XTAL/S
- C203: value 100uF/25V -> 100n; device resistor:CPOL-EUE5-10.5 -> resistor:C-EUC0603
- C301: value 22p -> 100n; device resistor:C-EUC0603 -> rcl:C-EUC0603
- C304: device resistor:C-EUC0603 -> rcl:C-EUC0603
- IC403: value MCP2515T-I/SO -> MAX481CPA; device microchip:MCP2515T-I/SO -> maxim:MAX481CPA
- IC404: value MCP2561-E/SN -> MAX481CPA; device microchip:MCP2561-E/SN -> maxim:MAX481CPA
- J601: value INPUT_PWR -> PANEL; device SparkFun-Connectors:M04-XH-RA -> SparkFun-Connectors:M08-XH-RA
- R403: value 120R -> 120
- R404: value 330R -> 120; device resistor:R-EU_R0603 -> rcl:R-EU_R0603
- U$7: value MOD_MEGA_LAYOUT_Z_ODD -> MOD_MEGA_LAYOUT_Y_EVEN; device encPhone:MOD_MEGA_LAYOUT_Z_ODD -> encPhone:MOD_MEGA_LAYOUT_Y_EVEN
- U$9: value MOD_MEGA_LAYOUT_Y_ODD -> MOD_MEGA_LAYOUT_Z_ODD; device encPhone:MOD_MEGA_LAYOUT_Y_ODD -> encPhone:MOD_MEGA_LAYOUT_Z_ODD
Connections:
- net MTR_RXD renamed MTR_PAN_RXD
- net MTR_TXD renamed MTR_PAN_TXD
- removed net !RESET1: C301.1, D301.A, IC301.PC6(/RESET), R301.1
- removed net CAN_CS: IC403.!CS
- removed net CAN_INT: IC403.!INT, LD401.C
- removed net FEED_RXD: IC301.PD0(RXD), U$6.14(TX3)
- removed net FEED_TXD: IC301.PD1(TXD), U$6.15(RX3)
- removed net N$21: C401.1, D401.A, IC403.!RESET, R405.1
- removed net N$22: C403.2, IC403.OSC1, Q401.1
- removed net N$23: C404.2, IC403.OSC2, Q401.2
- removed net N$24: LD401.A, R404.2
- removed net N$5: C303.2, IC301.PB7(XTAL2/TOSC2), Q301.1
- removed net P_FEED1: IC301.PD2(INT0), J612.3, R606.1
- removed net P_FEED2: IC301.PC5(ADC5/SCL), J612.2, R608.1
- removed net P_FEED3: IC301.PC4(ADC4/SDA), J612.1, R610.1
- removed net P_HALL1/A: J613.3, R605.1, R606.2
- removed net P_HALL2/B: J613.4, R607.1, R608.2
- removed net P_HALL3/Z: J613.5, R609.1, R610.2
- removed net P_VDD: J612.6, J613.6, R605.2, R607.2, R609.2
- removed net RX+: IC401G$1.A, J608.2, J609.2, R401.1
- removed net RX-: IC401G$1.B, J608.1, J609.1, R401.2
- removed net TX+: IC402G$1.A, J608.4, J609.4, R402.1
- removed net TX-: IC402G$1.B, J608.3, J609.3, R402.2
- removed net T_FEED1: IC301.PD3(INT1), J614.3, R616.1
- removed net T_FEED2: IC301.PC3(ADC3), J614.2, R614.1
- removed net T_FEED3: IC301.PC2(ADC2), J614.1, R612.1
- removed net T_HALL1/A: J615.3, R615.1, R616.2
- removed net T_HALL2/B: J615.4, R613.1, R614.2
- removed net T_HALL3/Z: J615.5, R611.1, R612.2
- removed net T_VDD: J614.6, J615.6, R611.2, R613.2, R615.2
- new net !CAN_CS: IC305.!CS, U$7.49
- new net +24V: C201.+, D201.C, J601.5, J601.6, J603.2, U201.IN+
- new net MTR_TILT_RXD: IC403G$1.DI, U$6.14(TX3)
- new net MTR_TILT_TXD: IC404G$1.RO, U$6.15(RX3)
- new net N$12: D604.C, J611.1
- new net N$13: C302.2, IC305.OSC1, X301.1
- new net PAN_RX+: IC401G$1.A, J608.2, R401.1
- new net PAN_RX-: IC401G$1.B, J608.1, R401.2
- new net PAN_TX+: IC402G$1.A, J608.4, R402.1
- new net PAN_TX-: IC402G$1.B, J608.3, R402.2
- new net P_RESV: D603.A, U$9.31
- new net RXD2: U$5.17(RX2), UART_RESV.1
- new net SCL: U$10.21(SCL)
- new net SDA: U$10.20(SDA)
- new net TILT_RX+: IC403G$1.A, J609.2, R403.1
- new net TILT_RX-: IC403G$1.B, J609.1, R403.2
- new net TILT_TX+: IC404G$1.A, J609.4, R404.1
- new net TILT_TX-: IC404G$1.B, J609.3, R404.2
- new net TXD2: U$5.16(TX2), UART_RESV.2
- new net T_RESV: D604.A, U$8.42
- net CAN_H: now also IC306.CAN_H, J601.1, J603.6, R306.2; no longer IC404.CAN_H, J602.1, J603.4, R403.2
- net CAN_L: now also IC306.CAN_L, J601.2, J603.5, R306.1; no longer IC404.CAN_L, J602.2, J603.3, R403.1
- net GND: now also C202.-, C203.2, C304.2, IC305.VSS, IC306.GND, IC306.STBY, IC404G$1.DE, IC404G$1.RE/, J607.4, UART_RESV.3; no longer C203.-, C204.2, C304.1, C305.2, C401.2, C402.2, C403.1, C404.1, IC301.GND@1, IC301.GND@2, IC403.VSS, IC404.GND, IC404.STBY, J607.1, J610.1, J611.1, J612.4, J612.5, J613.1, J613.2, J614.4, J614.5, J615.1, J615.2
- net MISO: now also IC305.SO; no longer IC403.SO
- net MOSI: now also IC305.SI; no longer IC403.SI
- net N$10: now also U$7.47; no longer J102.1, U$5.17(RX2)
- net N$11: now also D603.C, J610.1; no longer J102.2, U$5.16(TX2)
- net N$14: now also C303.2, IC305.OSC2, X301.2; no longer C304.2, IC301.AREF
- net N$6: now also R101.1, U$7.*13; no longer C302.2, IC301.PB6(XTAL1/TOSC1), Q301.2
- net N$9: now also C301.1, D301.A, IC305.!RESET, R305.1; no longer R101.1, U$7.31
- net P_ENABLE: now also U$9.33; no longer U$9.42
- net P_FAULT_RESET: now also U$9.35; no longer U$9.44*
- net P_HEALTH: now also U$9.37; no longer U$9.46*
- net P_HOME_SWITCH: now also J607.3, U$7.*11; no longer J607.2, U$7.33
- net RXCAN: now also IC305.RXCAN, IC306.RXD; no longer IC403.RXCAN, IC404.RXD
- net SCK: now also IC305.SCK; no longer IC403.SCK
- net TRIGGER_PWM: now also U$7.*45
- net TRIGGER_PWR_EN: now also U$7.43
- net TXCAN: now also IC305.TXCAN, IC306.TXD; no longer IC403.TXCAN, IC404.TXD
- net T_DOWN_LIM: now also J607.1, U$8.12*; no longer J607.4, U$7.37
- net T_ENABLE: now also U$8.44*; no longer U$9.48
- net T_FAULT_RESET: now also U$8.46*; no longer U$9.12*
- net T_HEALTH: now also U$8.48; no longer U$9.10*
- net T_UP_LIM: now also J607.2, U$8.10*; no longer J607.3, U$7.35
- net V+: no longer C601.+, D201.C, J601.1, J601.2, J603.6, U201.IN+
- net V-: now also C201.-, J601.7, J601.8, J603.1; no longer C601.-, J601.3, J601.4, J603.5
- net VCC: now also C202.+, C203.1, C304.1, IC305.VDD, IC306.VCC, IC403G$1.DE, IC403G$1.RE/, R305.2; no longer C203.+, C204.1, C305.1, C402.1, D401.C, IC301.AVCC, IC301.VCC, IC403.VDD, IC404.VCC, R301.2, R404.1, R405.2
- net VIDEO+: now also J601.3, J603.4; no longer J602.3, J603.2
- net VIDEO-: now also J601.4, J603.3; no longer J602.4, J603.1
Other:
- note added: "R403 & R404 optional"
- note removed: "PCINT10"
- note removed: "PCINT11"
- note removed: "PCINT12"
- note removed: "PCINT13"
- note removed: "PCINT18"
- note removed: "PCINT19"
